File: phototransmitter.kicad_sch (KiCad schematic)
At the start: 0 parts

Commit message: complete laser bias circuit
Parts:
- added C?: 10n, symbol Device:C
- added C?: 100u, symbol Device:C_Polarized
- added J?: SMA Laser, symbol Connector:Conn_Coaxial
- added Q? (x2): BC547, Package_TO_SOT_THT:TO-92_Inline, symbol Transistor_BJT:BC547
- added RV? (x2): 1M, symbol Device:R_Potentiometer
Connections:
- new net: Q?.1 (C), RV?.2 (x2)
- new net: J?.1 (In), Q?.3 (E), Q?.3 (E)
- new net +12V: C?.1, C?.2, RV?.1, RV?.1
- new net FPGA_TXn: Q?.2 (B)
- new net FPGA_TXp: Q?.2 (B)
- new net GND: C?.1, C?.2, J?.2 (Ext), RV?.3, RV?.3
