File: power_supply.kicad_sch (KiCad schematic)
At the start: 19 parts, among them J2 Conn_01x01_Male, J4 Conn_01x01_Male, U4 AP63203WU, U5 AP63205WU

Commit message: tweaked power circuit, sorted drc errors and warnings, visual checked pcb
Parts:
- J2: Source (none) -> https://onecall.farnell.com/multicomp/24-243-1/banana-socke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
- J4: Source (none) -> https://onecall.farnell.com/multicomp/24-243-2/receptacle-2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
Changed lines of the file:
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@@
+      (effects (font (size 1.27 1.27)) hide)
+    )
+    (property "Source" "https://onecall.farnell.com/multicomp/24-243-1/banana-socket-20a-4mm-pcb-red/dp/1698982?st=test%20connector" (id 4) (at 90.17 34.29 0)
       (effects (font (size 1.27 1.27)) hide)
     )
@@
       (effects (font (size 1.27 1.27)) hide)
     )
+    (property "Source" "https://onecall.farnell.com/multicomp/24-243-2/receptacle-20a-4mm-pcb-solder/dp/1698983?st=test%20connector" (id 4) (at 90.17 41.91 0)
+      (effects (font (size 1.27 1.27)) hide)
+    )

Commit message: Update sourcing URLs
Parts:
- JP5: Source (none) -> pcb
- U4: Source https://onecall.farnell.com/diodes-inc/ap63203wu-7/dc-dc-conv-sync-buck-1-1mhz-85deg/dp/3518307?ost=ap63203 -> https://onecall.farnell.com/diodes-inc/ap63203wu-7/dc-dc-conv-sync-buck-1-1mhz-85deg/dp/3518307
- U5: Source https://onecall.farnell.com/diodes-inc/ap63205wu-7/dc-dc-conv-sync-buck-1-1mhz-85deg/dp/3518308?st=ap63205 -> https://onecall.farnell.com/diodes-inc/ap63205wu-7/dc-dc-conv-sync-buck-1-1mhz-85deg/dp/3518308
Changed lines of the file:
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@@
       (effects (font (size 1.27 1.27)) hide)
     )
-    (property "Source" "https://onecall.farnell.com/diodes-inc/ap63205wu-7/dc-dc-conv-sync-buck-1-1mhz-85deg/dp/3518308?st=ap63205" (id 4) (at 139.7 104.14 0)
+    (property "Source" "https://onecall.farnell.com/diodes-inc/ap63205wu-7/dc-dc-conv-sync-buck-1-1mhz-85deg/dp/3518308" (id 4) (at 139.7 104.14 0)
       (effects (font (size 1.27 1.27)) hide)
     )
@@
       (effects (font (size 1.27 1.27)) hide)
     )
+    (property "Source" "pcb" (id 4) (at 160.02 34.29 0)
+      (effects (font (size 1.27 1.27)) hide)
+    )
     (pin "1")
     (pin "2")
@@
       (effects (font (size 1.27 1.27)) hide)
     )
-    (property "Source" "https://onecall.farnell.com/diodes-inc/ap63203wu-7/dc-dc-conv-sync-buck-1-1mhz-85deg/dp/3518307?ost=ap63203" (id 4) (at 139.7 66.04 0)
-      (effects (font (size 1.27 1.27)) hide)
-    )
+    (property "Source" "https://onecall.farnell.com/diodes-inc/ap63203wu-7/dc-dc-conv-sync-buck-1-1mhz-85deg/dp/3518307" (id 4) (at 139.7 66.04 0)
+      (effects (font (size 1.27 1.27)) hide)
+    )
