File: PHY.kicad_sch (KiCad schematic)
At the start: 50 parts, among them U1 LAN83C185-JT, Y1 25 MHz

Commit message: did lots of routing for phy
Parts:
- added D4: Green LED, LED_SMD:LED_1206_3216Metric_Pad1.42x1.75mm_HandSolder, symbol Device:LED
- added D5: Yellow LED, LED_SMD:LED_1206_3216Metric_Pad1.42x1.75mm_HandSolder, symbol Device:LED
Connections:
- net +3V3: no longer R18.1
- net PHY-VREG: now also R18.1
- net ETH-L1N: no longer names the net of R33.1
- net ETH-L1N: now also D4.1 (K)
- net ETH-L1P renamed PHY-AD1
- net PHY-AD1: now also D4.2 (A)
- net ETH-L2N: no longer names the net of R34.1
- net ETH-L2N: now also D5.1 (K)
- net ETH-L2P renamed PHY-AD2
- net PHY-AD2: now also D5.2 (A)
Changed lines of the file:
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@@
-    (stroke (width 0) (type default) (color 0 0 0 0))
-  )
-  (wire (pts (xy 55.88 114.3) (xy 55.88 110.49))
     (stroke (width 0) (type default) (color 0 0 0 0))
   )
@@
   )
   (wire (pts (xy 199.39 137.16) (xy 199.39 142.24))
-    (stroke (width 0) (type default) (color 0 0 0 0))
-  )
-  (wire (pts (xy 50.8 114.3) (xy 55.88 114.3))
     (stroke (width 0) (type default) (color 0 0 0 0))
   )
@@
     )
   )
-  (global_label "ETH-L2N" (shape input) (at 255.27 35.56 180) (fields_autoplaced)
-    (effects (font (size 1.27 1.27)) (justify right))
-    (property "Intersheet References" "${INTERSHEET_REFS}" (id 0) (at 244.2693 35.4806 0)
-      (effects (font (size 1.27 1.27)) (justify right) hide)
-    )
-  )
   (global_label "PHY-RX_ER" (shape input) (at 210.82 137.16 0) (fields_autoplaced)
     (effects (font (size 1.27 1.27)) (justify left))
@@
     )
   )
-  (global_label "ETH-L2P" (shape input) (at 255.27 27.94 180) (fields_autoplaced)
-    (effects (font (size 1.27 1.27)) (justify right))
-    (property "Intersheet References" "${INTERSHEET_REFS}" (id 0) (at 244.3298 27.8606 0)
-      (effects (font (size 1.27 1.27)) (justify right) hide)
-    )
-  )
-  (global_label "ETH-L1P" (shape input) (at 240.03 27.94 180) (fields_autoplaced)
-    (effects (font (size 1.27 1.27)) (justify right))
-    (property "Intersheet References" "${INTERSHEET_REFS}" (id 0) (at 229.0898 27.8606 0)
-      (effects (font (size 1.27 1.27)) (justify right) hide)
-    )
-  )
   (global_label "PHY-TX_CLK" (shape input) (at 222.25 119.38 0) (fields_autoplaced)
     (effects (font (size 1.27 1.27)) (justify left))
@@
     )
   )
+  (global_label "PHY-VREG" (shape input) (at 55.88 110.49 180) (fields_autoplaced)
+    (effects (font (size 1.27 1.27)) (justify right))
+    (property "Intersheet References" "${INTERSHEET_REFS}" (id 0) (at 43.4279 110.4106 0)
+      (effects (font (size 1.27 1.27)) (justify right) hide)
+    )
+  )
   (global_label "PHY-AD0" (shape input) (at 93.98 87.63 180) (fields_autoplaced)
     (effects (font (size 1.27 1.27)) (justify right))
@@
     (property "Intersheet References" "${INTERSHEET_REFS}" (id 0) (at 242.5036 102.7906 0)
       (effects (font (size 1.27 1.27)) (justify left) hide)
-    )
-  )
-  (global_label "ETH-L1N" (shape input) (at 240.03 35.56 180) (fields_autoplaced)
-    (effects (font (size 1.27 1.27)) (justify right))
-    (property "Intersheet References" "${INTERSHEET_REFS}" (id 0) (at 229.0293 35.4806 0)
-      (effects (font (size 1.27 1.27)) (justify right) hide)
     )
   )
@@
     (pin "2")
   )
+  (symbol (lib_id "Device:LED") (at 240.03 31.75 90) (unit 1)
+    (in_bom yes) (on_board yes) (fields_autoplaced)
+    (property "Reference" "D4" (id 0) (at 243.84 32.0674 90)
+      (effects (font (size 1.27 1.27)) (justify right))
+    )
+    (property "Value" "Green LED" (id 1) (at 243.84 34.6074 90)
+      (effects (font (size 1.27 1.27)) (justify right))
+    )
+    (property "Footprint" "LED_SMD:LED_1206_3216Metric_Pad1.42x1.75mm_HandSolder" (id 2) (at 240.03 31.75 0)
+      (effects (font (size 1.27 1.27)) hide)
+    )
+    (property "Datasheet" "~" (id 3) (at 240.03 31.75 0)
+      (effects (font (size 1.27 1.27)) hide)
+    )
+    (property "Source" "https://onecall.farnell.com/dialight/599-0281-007f/led-green-340mcd-525nm-1206/dp/3548452" (id 4) (at 240.03 31.75 0)
+      (effects (font (size 1.27 1.27)) hide)
+    )
+    (pin "1")
+    (pin "2")
+  )
   (symbol (lib_id "power:GND") (at 158.75 187.96 0) (unit 1)
     (in_bom yes) (on_board yes) (fields_autoplaced)
@@
     (pin "2")
   )
+  (symbol (lib_id "Device:LED") (at 255.27 31.75 90) (unit 1)
+    (in_bom yes) (on_board yes) (fields_autoplaced)
+    (property "Reference" "D5" (id 0) (at 259.08 32.0674 90)
+      (effects (font (size 1.27 1.27)) (justify right))
+    )
+    (property "Value" "Yellow LED" (id 1) (at 259.08 34.6074 90)
+      (effects (font (size 1.27 1.27)) (justify right))
+    )
+    (property "Footprint" "LED_SMD:LED_1206_3216Metric_Pad1.42x1.75mm_HandSolder" (id 2) (at 255.27 31.75 0)
+      (effects (font (size 1.27 1.27)) hide)
+    )
+    (property "Datasheet" "~" (id 3) (at 255.27 31.75 0)
+      (effects (font (size 1.27 1.27)) hide)
+    )
+    (property "Source" "https://onecall.farnell.com/dialight/599-0240-007f/led-yellow-126mcd-590nm-1206/dp/3548450?st=yellow" (id 4) (at 255.27 31.75 0)
+      (effects (font (size 1.27 1.27)) hide)
+    )
+    (pin "1")
+    (pin "2")
+  )
   (symbol (lib_id "Device:R") (at 45.72 57.15 90) (unit 1)
     (in_bom yes) (on_board yes) (fields_autoplaced)
@@
     (pin "2")
   )
-  (symbol (lib_id "power:+3V3") (at 50.8 114.3 0) (unit 1)
-    (in_bom yes) (on_board yes) (fields_autoplaced)
-    (property "Reference" "#PWR014" (id 0) (at 50.8 118.11 0)
-      (effects (font (size 1.27 1.27)) hide)
-    )
-    (property "Value" "+3V3" (id 1) (at 50.8 109.22 0))
-    (property "Footprint" "" (id 2) (at 50.8 114.3 0)
-      (effects (font (size 1.27 1.27)) hide)
-    )
-    (property "Datasheet" "" (id 3) (at 50.8 114.3 0)
-      (effects (font (size 1.27 1.27)) hide)
-    )
-    (pin "1")
-  )
   (symbol (lib_id "Device:C_Polarized") (at 19.05 153.67 0) (unit 1)
