File: laser.kicad_sch (KiCad schematic)
At the start: 17 parts, among them J3 Laser, Q1 BC547, Q2 BC547, U6 LM317_TO-220, U7 LM317_TO-220

Commit message: revised laser driver and power supplies
Parts:
- added D6, D7: 1N4148, Diode_THT:D_DO-35_SOD27_P7.62mm_Horizontal, symbol Diode:1N4148
- added R45, R47, R48, R49: 200R, Resistor_THT:R_Axial_DIN0207_L6.3mm_D2.5mm_P10.16mm_Horizontal, symbol Device:R
- R11, R2, R3, R4: value 240R -> 200R
Connections:
- net GND: now also Q1.3 (E), Q2.3 (E); no longer R11.1, R2.1, R3.1, R4.1
- net High volt: now also R11.2, R3.2; no longer Q1.1 (C)
- net Low volt: now also R45.2, R47.2, R48.2, R49.2; no longer Q2.1 (C), R11.2, R3.2
- new net: D7.2 (A), Q2.1 (C), R45.1, R47.1, R48.1, R49.1
- new net: D6.1 (K), D7.1 (K), J3.1
- new net: D6.2 (A), Q1.1 (C), R11.1, R2.1, R3.1, R4.1
Other:
- moved on the sheet: J3, Q1, Q2, R2, R4
